File: DBranded1/DBranded1.kicad_sch (KiCad schematic)
At the start: 6 parts, among them U1 NT3H2111W0FHKH

Commit message: bom and production files
Parts:
- R1: value 220 -> 1k
Changed lines of the file:
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@@
 			)
 		)
-		(property "Value" "220"
+		(property "Value" "1k"
 			(at 100.33 83.058 90)
 			(show_name no)
